File: hardware/reDIP-64-USB.kicad_sch (KiCad schematic)
At the start: 35 parts, among them J1 USB4080, Q1 PDTA143ZMB, U1 PTN5110NHQ, U2 LFE5UM5G-25F-8MG285C, U3 FUSB340, U4 DSC1103CE2-135.0000, U5 FSUSB42UMX

Commit message: A few improvements
* Changed MCLK pullup to 4.7k
* A few pin swaps for cleaner routing
* Example pin headers in BOM
* Replaced reduced lifetime "mobile only" capacitors
Parts:
- C1, C2, C3, C4: Notes 3.3V DC DERATED TO 1uF -> 3.3V DC DERATED TO 0.7uF; PN GRM035R60J475ME15D -> GRM033R60J225ME01D
Changed lines of the file:
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@@
   (title_block
     (title "reDIP 64")
-    (date "2022-04-10")
+    (date "2022-04-14")
     (rev "1.0")
     (company "Nimrod")
@@
       (effects (font (size 1.27 1.27)) hide)
     )
-    (property "Datasheet" "https://www.murata.com/products/productdetail.aspx?partno=GRM035R60J475ME15D" (id 3) (at 140.97 63.5 0)
-      (effects (font (size 1.27 1.27)) hide)
-    )
-    (property "Description" "CAP CER 4.7uF 6.3V 20% X5R 0201" (id 4) (at 140.97 63.5 0)
+    (property "Datasheet" "https://www.murata.com/products/productdetail.aspx?partno=GRM033R60J225ME01D" (id 3) (at 140.97 63.5 0)
+      (effects (font (size 1.27 1.27)) hide)
+    )
+    (property "Description" "CAP CER 2.2uF 6.3V 20% X5R 0201" (id 4) (at 140.97 63.5 0)
       (effects (font (size 1.27 1.27)) hide)
     )
@@
       (effects (font (size 1.27 1.27)) hide)
     )
-    (property "Notes" "3.3V DC DERATED TO 1uF" (id 6) (at 140.97 63.5 0)
-      (effects (font (size 1.27 1.27)) hide)
-    )
-    (property "PN" "GRM035R60J475ME15D" (id 7) (at 140.97 63.5 0)
+    (property "Notes" "3.3V DC DERATED TO 0.7uF" (id 6) (at 140.97 63.5 0)
+      (effects (font (size 1.27 1.27)) hide)
+    )
+    (property "PN" "GRM033R60J225ME01D" (id 7) (at 140.97 63.5 0)
       (effects (font (size 1.27 1.27)) hide)
     )
@@
       (effects (font (size 1.27 1.27)) hide)
     )
-    (property "Datasheet" "https://www.murata.com/products/productdetail.aspx?partno=GRM035R60J475ME15D" (id 3) (at 171.45 36.83 0)
-      (effects (font (size 1.27 1.27)) hide)
-    )
-    (property "Description" "CAP CER 4.7uF 6.3V 20% X5R 0201" (id 4) (at 171.45 36.83 0)
+    (property "Datasheet" "https://www.murata.com/products/productdetail.aspx?partno=GRM033R60J225ME01D" (id 3) (at 171.45 36.83 0)
+      (effects (font (size 1.27 1.27)) hide)
+    )
+    (property "Description" "CAP CER 2.2uF 6.3V 20% X5R 0201" (id 4) (at 171.45 36.83 0)
       (effects (font (size 1.27 1.27)) hide)
     )
@@
       (effects (font (size 1.27 1.27)) hide)
     )
-    (property "Notes" "3.3V DC DERATED TO 1uF" (id 6) (at 171.45 36.83 0)
-      (effects (font (size 1.27 1.27)) hide)
-    )
-    (property "PN" "GRM035R60J475ME15D" (id 7) (at 171.45 36.83 0)
+    (property "Notes" "3.3V DC DERATED TO 0.7uF" (id 6) (at 171.45 36.83 0)
+      (effects (font (size 1.27 1.27)) hide)
+    )
+    (property "PN" "GRM033R60J225ME01D" (id 7) (at 171.45 36.83 0)
       (effects (font (size 1.27 1.27)) hide)
     )
@@
       (effects (font (size 1.27 1.27)) hide)
     )
-    (property "Datasheet" "https://www.murata.com/products/productdetail.aspx?partno=GRM035R60J475ME15D" (id 3) (at 156.21 36.83 0)
-      (effects (font (size 1.27 1.27)) hide)
-    )
-    (property "Description" "CAP CER 4.7uF 6.3V 20% X5R 0201" (id 4) (at 156.21 36.83 0)
+    (property "Datasheet" "https://www.murata.com/products/productdetail.aspx?partno=GRM033R60J225ME01D" (id 3) (at 156.21 36.83 0)
+      (effects (font (size 1.27 1.27)) hide)
+    )
+    (property "Description" "CAP CER 2.2uF 6.3V 20% X5R 0201" (id 4) (at 156.21 36.83 0)
       (effects (font (size 1.27 1.27)) hide)
     )
@@
       (effects (font (size 1.27 1.27)) hide)
     )
-    (property "Notes" "3.3V DC DERATED TO 1uF" (id 6) (at 156.21 36.83 0)
-      (effects (font (size 1.27 1.27)) hide)
-    )
-    (property "PN" "GRM035R60J475ME15D" (id 7) (at 156.21 36.83 0)
+    (property "Notes" "3.3V DC DERATED TO 0.7uF" (id 6) (at 156.21 36.83 0)
+      (effects (font (size 1.27 1.27)) hide)
+    )
+    (property "PN" "GRM033R60J225ME01D" (id 7) (at 156.21 36.83 0)
       (effects (font (size 1.27 1.27)) hide)
     )
@@
       (effects (font (size 1.27 1.27)) hide)
     )
-    (property "Datasheet" "https://www.murata.com/products/productdetail.aspx?partno=GRM035R60J475ME15D" (id 3) (at 181.61 36.83 0)
-      (effects (font (size 1.27 1.27)) hide)
-    )
-    (property "Description" "CAP CER 4.7uF 6.3V 20% X5R 0201" (id 4) (at 181.61 36.83 0)
+    (property "Datasheet" "https://www.murata.com/products/productdetail.aspx?partno=GRM033R60J225ME01D" (id 3) (at 181.61 36.83 0)
+      (effects (font (size 1.27 1.27)) hide)
+    )
+    (property "Description" "CAP CER 2.2uF 6.3V 20% X5R 0201" (id 4) (at 181.61 36.83 0)
       (effects (font (size 1.27 1.27)) hide)
     )
@@
       (effects (font (size 1.27 1.27)) hide)
     )
-    (property "Notes" "3.3V DC DERATED TO 1uF" (id 6) (at 181.61 36.83 0)
-      (effects (font (size 1.27 1.27)) hide)
-    )
-    (property "PN" "GRM035R60J475ME15D" (id 7) (at 181.61 36.83 0)
-      (effects (font (size 1.27 1.27)) hide)
-    )
+    (property "Notes" "3.3V DC DERATED TO 0.7uF" (id 6) (at 181.61 36.83 0)
+      (effects (font (size 1.27 1.27)) hide)
+    )
+    (property "PN" "GRM033R60J225ME01D" (id 7) (at 181.61 36.83 0)
+      (effects (font (size 1.27 1.27)) hide)
+    )

Commit message: Audio upgrade
* Changed from line out to headphone out with 10uF tantalum capacitors
* PTN5110 decoupling capacitor QA
Parts:
- C1: footprint Capacitor_SMD:C_0201_0603Metric -> Capacitor_SMD:C_0402_1005Metric; Notes 3.3V DC DERATED TO 0.7uF -> 5V DC DERATED TO 1uF; PN GRM033R60J225ME01D -> GRM155R61E225ME11D
- C3: Notes 3.3V DC DERATED TO 0.7uF -> 5V DC DERATED TO 0.6uF; PN GRM033R60J225ME01D -> GRM035R61A225ME01D
